Commit message: Fixed constraint error, simple example works

File: assets/servo/Servo.urdf (robot description, URDF)
Before this commit: robot Servo, 2 links, 1 joints
Joints:
- joint Joint: limit lower=-1.57 upper=1.57 effort=1.5 velocity=3.0 -> lower=-1.57 upper=1.57 effort=1.5 velocity=6.0

Commit message: Fixed servo parameters following Dynamixel AX-18

File: assets/servo/Servo.urdf (robot description, URDF)
Before this commit: robot Servo, 2 links, 1 joints
Joints:
- joint Joint: limit lower=-1.57 upper=1.57 effort=1.5 velocity=6.0 -> lower=-1.57 upper=1.57 effort=1.8 velocity=10.6
