Commit message: Changed environment reset to avoid collision with plane
Using `saveState` and `restoreState` doesn't do that much for our use
case so to save some time we simply run `setup` again. This has the
added benefit that it avoids the root module colliding with the plane.

File: assets/plane/plane.urdf (robot description, URDF)
Before this commit: robot plane, 1 links, 0 joints
Links:
- link planeLink: geometry collision box size=30 30 0.001; visual mesh filename=plane.obj scale=1 1 1
